Commit message: Robot Bouge 05 fevrirer

File: catkin_ws/src/robot_description/urdf/robot.urdf (robot description, URDF)
Before this commit: robot robot, 10 links, 9 joints
Links:
- removed link end_effector
- added link end_effector_base, mass 1.0; collision box size=0.05 .02 .01; visual box size=0.05 .02 .01
- added link end_effector_left, mass 1.0; collision box size=0.005 .02 .02; visual box size=.02 .02 0.005
- added link end_effector_right, mass 1.0; collision box size=0.005 .02 .02; visual box size=.02 .02 0.005
Joints:
- added joint joint5: type prismatic, parent end_effector_base, child end_effector_right, origin xyz=-0.025 0 0.125 rpy=0 1.57 0, axis 0 0 1, limit lower=0 upper=.02 effort=100 velocity=3
- added joint joint6: type prismatic, parent end_effector_base, child end_effector_left, origin xyz=0.025 0 0.125 rpy=0 -1.57 0, axis 0 0 1, limit lower=0 upper=.02 effort=100 velocity=3
- joint joint2: limit lower=-1.5707963267948 upper=1.5707963267948 effort=10 velocity=3 -> lower=-3.14 upper=3.14 effort=10 velocity=3
- joint joint3: limit lower=-.08 upper=.08 effort=10 velocity=3 -> lower=-.08 upper=.08 effort=100 velocity=3
- joint joint4: child end_effector -> end_effector_base
- joint joint_arm_endarm_2: limit (none) -> lower=-3 upper=3 effort=10 velocity=3
